File: Arduino UNO.kicad_pcb (KiCad board)
At the start: 2 copper layers, 100.1 x 75.9 mm, 56 parts, among them J1 M20-9980345, J2 M20-9980245, J3 M20-9980345, J4 PPTC101LFBN-RC, J5 PPTC081LFBN-RC, J6 PPTC061LFBN-RC, J7 PPTC081LFBN-RC, J8 USB_C_Receptacle_USB2.0_16P, J9 PJ-102AH, Q1 FDN340P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

Commit message: updated logos
Parts:
- added REF**: MountingHole_3.2mm_M3, MountingHole:MountingHole_3.2mm_M3, F.Cu at (211.5, 139.0)
- added REF**: MountingHole_3.2mm_M3, MountingHole:MountingHole_3.2mm_M3, F.Cu at (129.5, 139.0)
- added REF**: MountingHole_3.2mm_M3, MountingHole:MountingHole_3.2mm_M3, F.Cu at (129.5, 70.0)
- added REF**: MountingHole_3.2mm_M3, MountingHole:MountingHole_3.2mm_M3, F.Cu at (211.5, 70.0)
